File: kicad/circuit/circuit.kicad_pcb (KiCad board)
At the start: 2 copper layers, 49.7 x 53.1 mm, 23 parts, among them J1 4X4 Matrix, J1.1 2X2 Matrix A, J1.1.1 Button 1, J1.1.2 Button 2, J1.1.3 Button 5, J1.1.4 Button 6, J1.2 2X2 Matrix B, J1.2.1 Button 3, J1.2.2 Button 4, J1.3 2X2 Matrix C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

Commit message: add i2c header
Parts:
- added J3: I2C, Connector_PinHeader_2.54mm:PinHeader_2x02_P2.54mm_Vertical_SMD, F.Cu at (222.0, 84.0)
- moved C3 1.94 mm to (238.8, 72.5)
- renumbered J3 to J2
Routing:
- net /SDA: track 7.61 -> 85.6 mm, vias 0 -> 1
- net /SCL: track 7.15 -> 82.1 mm, vias 0 -> 1
- net /R2: track 178.0 -> 193.1 mm
- net /R4: track 54.2 -> 66.3 mm
- net /R3: track 65.1 -> 72.4 mm
- net /L2: track 96.7 -> 101.9 mm
- net /L1: track 147.1 -> 151.4 mm
- net +5V: track 4.53 -> 3.34 mm, vias 2 -> 3
- net /R1: track 150.9 -> 151.8 mm

Commit message: add joystick connecting over rj45
Parts:
- removed SW1: Reset, Button_Switch_SMD:SW_Push_1P1T_NO_6x6mm_H9.5mm
- added J5: Joystick, Connector_PinHeader_2.54mm:PinHeader_2x03_P2.54mm_Vertical_SMD, F.Cu at (245.9, 72.9)
- moved J1 1.23 mm to (222.1, 57.3)
Connections:
- J4 pad 4: +5V -> /RX
- J4 pad 6: /SDA -> /RY
- J4 pad 8: /SCL -> /Switch
Routing:
- net /Switch: track 0.00 -> 21.6 mm, vias 0 -> 2
- net /RY: track 0.00 -> 19.6 mm, vias 0 -> 2
- net /RX: track 0.00 -> 18.2 mm
- net /L2: track 101.9 -> 104.6 mm
- net /L1: track 151.4 -> 153.6 mm
- net /RESET: track 57.5 -> 55.4 mm
- net /L4: track 81.7 -> 83.2 mm
- net +5V: track 3.34 -> 2.07 mm, vias 3 -> 4
- net /L3: track 92.1 -> 93.4 mm
- net /R3: track 72.4 -> 73.6 mm
- net /R4: track 66.3 -> 67.5 mm
- net /R1: track 151.8 -> 153.0 mm

Commit message: update pcb and documentation
Parts:
- C3: value 100 µF -> 10 µF; footprint Capacitor_SMD:C_0402_1005Metric -> Capacitor_SMD:C_1206_3216Metric
- moved C3 14.5 mm to (225.3, 67.3), turned to 0 degrees
Routing:
- net /SCL: track 82.3 -> 86.9 mm
- net /SDA: track 85.5 -> 89.9 mm
- net +5V: track 2.07 -> 2.61 mm
