File: kicad/circuit/circuit.kicad_sch (KiCad schematic)
At the start: 19 parts, among them J1 4X4 Matrix, J1.1 2X2 Matrix A, J1.1.1 Button 1, J1.1.2 Button 2, J1.1.3 Button 5, J1.1.4 Button 6, J1.2 2X2 Matrix B, J1.2.1 Button 3, J1.2.2 Button 4, J1.3 2X2 Matrix C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

Commit message: add i2c header
Parts:
- added J3: I2C, Connector_PinHeader_2.54mm:PinHeader_2x02_P2.54mm_Vertical_SMD, symbol Connector:Conn_01x04_Pin
- renumbered J3 to J2
Connections:
- net +5V: now also J3.2 (Pin_2)
- net GND: now also J3.1 (Pin_1)
- net SCL: now also J3.4 (Pin_4)
- net SDA: now also J3.3 (Pin_3)
Changed lines of the file:
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@@
+	)
+	(junction
+		(at 121.92 90.17)
+		(diameter 0)
+		(color 0 0 0 0)
 	)
 	(junction
@@
 	)
 	(junction
+		(at 121.92 95.25)
+		(diameter 0)
+		(color 0 0 0 0)
+	)
+	(junction
 		(at 138.43 100.33)
 		(diameter 0)
@@
 	)
 	(junction
+		(at 121.92 97.79)
+		(diameter 0)
+		(color 0 0 0 0)
+	)
+	(junction
 		(at 115.57 113.03)
 		(diameter 0)
@@
 	)
 	(junction
+		(at 121.92 92.71)
+		(diameter 0)
+		(color 0 0 0 0)
+	)
+	(junction
 		(at 66.04 53.34)
 		(diameter 0)
@@
 	(wire
 		(pts
-			(xy 106.68 90.17) (xy 133.35 90.17)
+			(xy 106.68 90.17) (xy 121.92 90.17)
+		)
+		(stroke
+			(width 0)
+			(type default)
+		)
+	)
+	(wire
+		(pts
+			(xy 121.92 90.17) (xy 133.35 90.17)
 		)
 		(stroke
@@
 	(wire
 		(pts
+			(xy 121.92 95.25) (xy 138.43 95.25)
+		)
+		(stroke
+			(width 0)
+			(type default)
+		)
+	)
+	(wire
+		(pts
 			(xy 132.08 165.1) (xy 109.22 165.1)
 		)
@@
 	(wire
 		(pts
+			(xy 121.92 97.79) (xy 134.62 97.79)
+		)
+		(stroke
+			(width 0)
+			(type default)
+		)
+	)
+	(wire
+		(pts
 			(xy 120.65 64.77) (xy 123.19 64.77)
 		)
@@
 	(wire
 		(pts
+			(xy 121.92 90.17) (xy 121.92 91.44)
+		)
+		(stroke
+			(width 0)
+			(type default)
+		)
+	)
+	(wire
+		(pts
 			(xy 115.57 107.95) (xy 115.57 113.03)
 		)
@@
 	(wire
 		(pts
-			(xy 81.28 97.79) (xy 134.62 97.79)
+			(xy 81.28 97.79) (xy 121.92 97.79)
 		)
 		(stroke
@@
 	(wire
 		(pts
+			(xy 121.92 92.71) (xy 121.92 93.98)
+		)
+		(stroke
+			(width 0)
+			(type default)
+		)
+	)
+	(wire
+		(pts
 			(xy 81.28 107.95) (xy 86.36 107.95)
 		)
@@
 	(wire
 		(pts
-			(xy 81.28 95.25) (xy 138.43 95.25)
+			(xy 81.28 95.25) (xy 121.92 95.25)
 		)
 		(stroke
@@
 	(wire
 		(pts
+			(xy 121.92 97.79) (xy 121.92 99.06)
+		)
+		(stroke
+			(width 0)
+			(type default)
+		)
+	)
+	(wire
+		(pts
+			(xy 121.92 92.71) (xy 138.43 92.71)
+		)
+		(stroke
+			(width 0)
+			(type default)
+		)
+	)
+	(wire
+		(pts
 			(xy 91.44 40.64) (xy 99.06 40.64)
 		)
@@
 	(wire
 		(pts
-			(xy 101.6 92.71) (xy 138.43 92.71)
+			(xy 101.6 92.71) (xy 121.92 92.71)
 		)
 		(stroke
@@
 		(pts
 			(xy 114.3 121.92) (xy 132.08 121.92)
+		)
+		(stroke
+			(width 0)
+			(type default)
+		)
+	)
+	(wire
+		(pts
+			(xy 121.92 95.25) (xy 121.92 96.52)
 		)
 		(stroke
@@
 		(on_board yes)
 		(dnp no)
-		(property "Reference" "J3"
+		(property "Reference" "J2"
 			(at 118.11 38.0999 0)
 			(effects
@@
 			(project ""
 				(path "/edf5049a-0fa6-4e51-97b2-c2c53b61158b"
-					(reference "J3")
+					(reference "J2")
 					(unit 1)
 				)
@@
 					(unit 1)
 				)
+			)
+		)
+	)
+	(symbol
+		(lib_id "Connector:Conn_01x04_Pin")
+		(at 116.84 93.98 0)
+		(unit 1)
+		(exclude_from_sim no)
+		(in_bom yes)
+		(on_board yes)
+		(dnp no)
+		(fields_autoplaced yes)
+		(property "Reference" "J3"
+			(at 117.475 86.36 0)
+			(effects
+				(font
+					(size 1.27 1.27)
+				)
+			)
+		)
+		(property "Value" "I2C"
+			(at 117.475 88.9 0)
+			(effects
+				(font
+					(size 1.27 1.27)
+				)
+			)
+		)
+		(property "Footprint" "Connector_PinHeader_2.54mm:PinHeader_2x02_P2.54mm_Vertical_SMD"
+			(at 116.84 93.98 0)
+			(effects
+				(font
+					(size 1.27 1.27)
+				)
+				(hide yes)
+			)
+		)
+		(property "Datasheet" "~"
+			(at 116.84 93.98 0)
+			(effects
+				(font
+					(size 1.27 1.27)
+				)
+				(hide yes)
+			)
+		)
+		(property "Description" "Generic connector, single row, 01x04, script generated"
+			(at 116.84 93.98 0)
+			(effects
+				(font
+					(size 1.27 1.27)
+				)
+				(hide yes)
+			)
+		)
+		(pin "1"
+		)
+		(pin "4"
+		)
+		(pin "3"
+		)
+		(pin "2"
+		)
+		(instances
+			(project ""
+				(path "/edf5049a-0fa6-4e51-97b2-c2c53b61158b"
+					(reference "J3")
+					(unit 1)
+				)

Commit message: add joystick connecting over rj45
Parts:
- removed SW1: Reset, Button_Switch_SMD:SW_Push_1P1T_NO_6x6mm_H9.5mm, symbol Switch:SW_Push
- added J5: Joystick, Connector_PinHeader_2.54mm:PinHeader_2x03_P2.54mm_Vertical_SMD, symbol Connector:Conn_01x05_Pin
Connections:
- net +5V: now also J5.2 (Pin_2); no longer J4.4
- net GND: now also J5.1 (Pin_1)
- net SCL: no longer J4.8
- net SDA: no longer J4.6
- new net RX: J4.4, J5.3 (Pin_3)
- new net RY: J4.6, J5.4 (Pin_4)
- new net Switch: J4.8, J5.5 (Pin_5)
Other:
- moved on the sheet: J4

Commit message: update pcb and documentation
Parts:
- C3: value 100 µF -> 10 µF; footprint Capacitor_SMD:C_0402_1005Metric -> Capacitor_SMD:C_1206_3216Metric
Changed lines of the file:
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@@
 			)
 		)
-		(property "Value" "100 µF"
+		(property "Value" "10 µF"
 			(at 35.56 88.8935 0)
 			(effects
@@
 			)
 		)
-		(property "Footprint" "Capacitor_SMD:C_0402_1005Metric"
+		(property "Footprint" "Capacitor_SMD:C_1206_3216Metric"
 			(at 33.02 87.63 0)
 			(effects
